File: 2can_filter.sch (KiCad schematic (older format))
At the start: 19 parts, among them J3 USB mini-B SMD, J4 NOT_FITTED_SWD_Conn_01x04_Male, U5 STM32F105RBTx, U6 TJA1040T, U7 TJA1040T, Y1 Crystal KX-7 25MHz

Commit message: add missed footprints, add additional capasitors on 3.3V line, fix banch of ERC errors
Parts:
- removed R3, R4: 10k, Resistors_SMD:R_0805, symbol R
- removed Y1: Crystal KX-7 25MHz, symbol Crystal
- added Y1: Crystal KX-13 25MHz, Crystals:Crystal_SMD_7050-4pin_7.0x5.0mm, symbol Crystal_GND24
- C21: renamed from C9; value 12pF -> 16pF
- C22: renamed from C10; value 12pF -> 16pF
- renumbered C11 to C23, C12 to C24
Connections:
- wire segments 77 -> 82
Changed lines of the file:
@@
 	1500 6500 1950 6500
 $Comp
-L C C11
+L C C23
 U 1 1 5A09EB1A
 P 10900 4450
-F 0 "C11" H 10925 4550 50  0000 L CNN
+F 0 "C23" H 10925 4550 50  0000 L CNN
 F 1 "10pF" H 10925 4350 50  0000 L CNN
 F 2 "Capacitors_SMD:C_0805" H 10938 4300 50  0001 C CNN
@@
 +3V3
 $Comp
-L GND #PWR14
+L GND #PWR020
 U 1 1 5A09EB1D
 P 1750 6600
-F 0 "#PWR14" H 1750 6350 50  0001 C CNN
+F 0 "#PWR020" H 1750 6350 50  0001 C CNN
 F 1 "GND" H 1750 6450 50  0000 C CNN
 F 2 "" H 1750 6600 50  0001 C CNN
@@
 Connection ~ 4800 5000
 $Comp
-L GND #PWR15
+L GND #PWR021
 U 1 1 5A09EB1E
 P 4900 5100
-F 0 "#PWR15" H 4900 4850 50  0001 C CNN
+F 0 "#PWR021" H 4900 4850 50  0001 C CNN
 F 1 "GND" H 4900 4950 50  0000 C CNN
 F 2 "" H 4900 5100 50  0001 C CNN
@@
 Connection ~ 10900 4150
 $Comp
-L C C12
+L C C24
 U 1 1 5A09EB1F
 P 10900 5850
-F 0 "C12" H 10925 5950 50  0000 L CNN
+F 0 "C24" H 10925 5950 50  0000 L CNN
 F 1 "10pF" H 10925 5750 50  0000 L CNN
 F 2 "Capacitors_SMD:C_0805" H 10938 5700 50  0001 C CNN
@@
 Wire Wire Line
 	8800 3950 9300 3950
-$Comp
-L R R3
-U 1 1 5A048BC2
-P 9200 4600
-F 0 "R3" V 9280 4600 50  0000 C CNN
-F 1 "10k" V 9200 4600 50  0000 C CNN
-F 2 "Resistors_SMD:R_0805" V 9130 4600 50  0001 C CNN
-F 3 "" H 9200 4600 50  0001 C CNN
-	1    9200 4600
-	-1   0    0    1
-$EndComp
-Wire Wire Line
-	9200 4450 9200 4350
+Wire Wire Line
+	9200 4350 9200 4600
 Wire Wire Line
 	9200 4350 9300 4350
-Wire Wire Line
-	9200 4750 9200 4800
-$Comp
-L GND #PWR20
+$Comp
+L GND #PWR022
 U 1 1 5A048D0B
 P 9800 4650
-F 0 "#PWR20" H 9800 4400 50  0001 C CNN
+F 0 "#PWR022" H 9800 4400 50  0001 C CNN
 F 1 "GND" H 9800 4500 50  0000 C CNN
 F 2 "" H 9800 4650 50  0001 C CNN
@@
 	9800 4550 9800 4650
 $Comp
-L GND #PWR22
+L GND #PWR023
 U 1 1 5A09EB24
 P 10900 4650
-F 0 "#PWR22" H 10900 4400 50  0001 C CNN
+F 0 "#PWR023" H 10900 4400 50  0001 C CNN
 F 1 "GND" H 10900 4500 50  0000 C CNN
 F 2 "" H 10900 4650 50  0001 C CNN
@@
 Wire Wire Line
 	10900 4650 10900 4600
-$Comp
-L GND #PWR18
-U 1 1 5A09EB25
-P 9200 4800
-F 0 "#PWR18" H 9200 4550 50  0001 C CNN
-F 1 "GND" H 9200 4650 50  0000 C CNN
-F 2 "" H 9200 4800 50  0001 C CNN
-F 3 "" H 9200 4800 50  0001 C CNN
-	1    9200 4800
-	1    0    0    -1
-$EndComp
-$Comp
-L R R4
-U 1 1 5A09EB26
-P 9200 6000
-F 0 "R4" V 9280 6000 50  0000 C CNN
-F 1 "10k" V 9200 6000 50  0000 C CNN
-F 2 "Resistors_SMD:R_0805" V 9130 6000 50  0001 C CNN
-F 3 "" H 9200 6000 50  0001 C CNN
-	1    9200 6000
-	-1   0    0    1
-$EndComp
-Wire Wire Line
-	9200 5850 9200 5750
 Wire Wire Line
 	9200 5750 9300 5750
-Wire Wire Line
-	9200 6150 9200 6200
-$Comp
-L GND #PWR19
-U 1 1 5A09EB27
-P 9200 6200
-F 0 "#PWR19" H 9200 5950 50  0001 C CNN
-F 1 "GND" H 9200 6050 50  0000 C CNN
-F 2 "" H 9200 6200 50  0001 C CNN
-F 3 "" H 9200 6200 50  0001 C CNN
-	1    9200 6200
-	1    0    0    -1
-$EndComp
-$Comp
-L GND #PWR21
+$Comp
+L GND #PWR024
 U 1 1 5A09EB28
 P 9800 6050
-F 0 "#PWR21" H 9800 5800 50  0001 C CNN
+F 0 "#PWR024" H 9800 5800 50  0001 C CNN
 F 1 "GND" H 9800 5900 50  0000 C CNN
 F 2 "" H 9800 6050 50  0001 C CNN
@@
 	9800 5950 9800 6050
 $Comp
-L GND #PWR23
+L GND #PWR025
 U 1 1 5A0491F4
 P 10900 6100
-F 0 "#PWR23" H 10900 5850 50  0001 C CNN
+F 0 "#PWR025" H 10900 5850 50  0001 C CNN
 F 1 "GND" H 10900 5950 50  0000 C CNN
 F 2 "" H 10900 6100 50  0001 C CNN
@@
 	8750 2950 8750 2800
 $Comp
-L GND #PWR17
+L GND #PWR026
 U 1 1 5A0498E0
 P 8750 2950
-F 0 "#PWR17" H 8750 2700 50  0001 C CNN
+F 0 "#PWR026" H 8750 2700 50  0001 C CNN
 F 1 "GND" H 8750 2800 50  0000 C CNN
 F 2 "" H 8750 2950 50  0001 C CNN
@@
 Connection ~ 2600 6500
 $Comp
-L Crystal Y1
-U 1 1 5A04A56A
-P 1350 3150
-F 0 "Y1" H 1350 3300 50  0000 C CNN
-F 1 "Crystal KX-7 25MHz" H 1300 3450 50  0000 C CNN
-F 2 "" H 1350 3150 50  0001 C CNN
-F 3 "" H 1350 3150 50  0001 C CNN
-	1    1350 3150
-	1    0    0    -1
-$EndComp
-$Comp
-L C C10
+L C C22
 U 1 1 5A04A61B
 P 1650 3400
-F 0 "C10" H 1675 3500 50  0000 L CNN
-F 1 "12pF" H 1675 3300 50  0000 L CNN
+F 0 "C22" H 1675 3500 50  0000 L CNN
+F 1 "16pF" H 1675 3300 50  0000 L CNN
 F 2 "Capacitors_SMD:C_0805" H 1688 3250 50  0001 C CNN
 F 3 "" H 1650 3400 50  0001 C CNN
@@
 $EndComp
 $Comp
-L C C9
+L C C21
 U 1 1 5A04A6A5
 P 1050 3400
-F 0 "C9" H 1075 3500 50  0000 L CNN
-F 1 "12pF" H 1075 3300 50  0000 L CNN
+F 0 "C21" H 1075 3500 50  0000 L CNN
+F 1 "16pF" H 1075 3300 50  0000 L CNN
 F 2 "Capacitors_SMD:C_0805" H 1088 3250 50  0001 C CNN
 F 3 "" H 1050 3400 50  0001 C CNN
@@
 $EndComp
 $Comp
-L GND #PWR12
+L GND #PWR027
 U 1 1 5A04A703
 P 1050 3650
-F 0 "#PWR12" H 1050 3400 50  0001 C CNN
+F 0 "#PWR027" H 1050 3400 50  0001 C CNN
 F 1 "GND" H 1050 3500 50  0000 C CNN
 F 2 "" H 1050 3650 50  0001 C CNN
@@
 $EndComp
 $Comp
-L GND #PWR13
+L GND #PWR028
 U 1 1 5A04A747
 P 1650 3650
-F 0 "#PWR13" H 1650 3400 50  0001 C CNN
+F 0 "#PWR028" H 1650 3400 50  0001 C CNN
 F 1 "GND" H 1650 3500 50  0000 C CNN
 F 2 "" H 1650 3650 50  0001 C CNN
@@
 Connection ~ 1650 3150
 $Comp
-L GND #PWR16
+L GND #PWR029
 U 1 1 5A04B0EB
-P 5750 6500
-F 0 "#PWR16" H 5750 6250 50  0001 C CNN
-F 1 "GND" H 5750 6350 50  0000 C CNN
-F 2 "" H 5750 6500 50  0001 C CNN
-F 3 "" H 5750 6500 50  0001 C CNN
-	1    5750 6500
+P 5750 6550
+F 0 "#PWR029" H 5750 6300 50  0001 C CNN
+F 1 "GND" H 5750 6400 50  0000 C CNN
+F 2 "" H 5750 6550 50  0001 C CNN
+F 3 "" H 5750 6550 50  0001 C CNN
+	1    5750 6550
 	1    0    0    -1
 $EndComp
@@
 	5650 6400 5750 6400
 Wire Wire Line
-	5750 6400 5750 6500
+	5750 6400 5750 6550
 $Comp
 L R R2
@@
 Wire Wire Line
 	4100 6500 4000 6500
+$Comp
+L Crystal_GND24 Y1
+U 1 1 5A0DDD49
+P 1350 3150
+F 0 "Y1" H 1475 3350 50  0000 L CNN
+F 1 "Crystal KX-13 25MHz" H 1475 3275 50  0000 L CNN
+F 2 "Crystals:Crystal_SMD_7050-4pin_7.0x5.0mm" H 1350 3150 50  0001 C CNN
+F 3 "" H 1350 3150 50  0001 C CNN
+	1    1350 3150
+	1    0    0    -1
+$EndComp
+Wire Wire Line
+	1350 2950 850  2950
+Wire Wire Line
+	850  2950 850  3600
+Wire Wire Line
+	850  3600 1350 3600
+Connection ~ 1050 3600
+Wire Wire Line
+	1350 3600 1350 3350
+Wire Wire Line
+	5650 6500 5750 6500
+Connection ~ 5750 6500
+Wire Wire Line
+	9200 4600 9800 4600
+Connection ~ 9800 4600
+Wire Wire Line
+	9800 6000 9200 6000
+Connection ~ 9800 6000
+Wire Wire Line
+	9200 6000 9200 5750
 $EndSCHEMATC

Commit message: add footprints to SWD connectors
Parts:
- J4: footprint (none) -> Pin_Headers:Pin_Header_Straight_1x04_Pitch2.54mm
Changed lines of the file:
@@
 F 0 "J4" H 8950 2900 50  0000 C CNN
 F 1 "NOT_FITTED_SWD_Conn_01x04_Male" H 8750 2300 50  0000 C CNN
-F 2 "" H 8950 2700 50  0001 C CNN
+F 2 "Pin_Headers:Pin_Header_Straight_1x04_Pitch2.54mm" H 8950 2700 50  0001 C CNN
 F 3 "" H 8950 2700 50  0001 C CNN
 	1    8950 2700

Commit message: change usb fp
Parts:
- J3: footprint 54819-0572:MOLEXMINIBTYPEB_1 -> zulljon:USB_mini_B
Changed lines of the file:
@@
 F 0 "J3" H 5150 6450 50  0000 C CNN
 F 1 "USB mini-B SMD" H 5250 5950 50  0000 C CNN
-F 2 "54819-0572:MOLEXMINIBTYPEB_1" H 5150 5850 50  0001 C CNN
+F 2 "zulljon:USB_mini_B" H 5150 5850 50  0001 C CNN
 F 3 "http://www.molex.com/webdocs/datasheets/pdf/en-us/0548190572_IO_CONNECTORS.pdf" H 5150 5750 50  0001 C CNN
 F 4 "Surface mount onthego connector,1A 30V Molex On-The-Go Series Right Angle SMT Version 2.0 Type B Mini USB Connector Receptacle, 30 V, 1A" H 5150 5650 50  0001 C CNN "Description"

Commit message: rescue the stm32 mcu_s, add pcb list info
Parts:
- U5: symbol STM32F105RBTx -> STM32F105RBTx-RESCUE-instrument_cluster
Changed lines of the file:
@@
 EESchema Schematic File Version 2
+LIBS:instrument_cluster-rescue
 LIBS:power
 LIBS:device
@@
 $EndDescr
 $Comp
-L STM32F105RBTx U5
+L STM32F105RBTx-RESCUE-instrument_cluster U5
 U 1 1 5A09EB17
 P 4900 2900
